Commit message: correct homing added

File: urdf/legs.urdf (robot description, URDF)
Before this commit: robot legs, 25 links, 24 joints
Links:
- removed link trunk_interia
- added link base; visual box size=0.3 0.2 0.093
- link trunk: mass None -> 3.3; geometry collision box size=0.216 0.098 0.048; visual box size=0.20 0.10 0.096
Joints:
- removed joint trunk_to_trunk_interia
- added joint floating_base: type fixed, parent base, child trunk, origin xyz=0 0 0 rpy=0 0 0
- joint FL_calf_joint: origin xyz=0 0 -0.2115 rpy=0 0 0 -> xyz=0 0.07125 -0.21183 rpy=0 -0.98 0
- joint FL_foot_fixed: origin xyz=0 0 -0.23039 rpy=0 0 0 -> xyz=0 0 -0.240 rpy=0 0 0
- joint FL_thigh_joint: origin xyz=0 0.077476 0 rpy=0 0 0 -> xyz=0.06 0.015 0 rpy=0 0 0
- joint FR_calf_joint: origin xyz=0 0 -0.2115 rpy=0 0 0 -> xyz=0 -0.07125 -0.21183 rpy=0 -0.98 0
- joint FR_foot_fixed: origin xyz=0 0 -0.23039 rpy=0 0 0 -> xyz=0 0 -0.240 rpy=0 0 0
- joint FR_thigh_joint: origin xyz=0 -0.077476 0 rpy=0 0 0 -> xyz=0.06 -0.015 0 rpy=0 0 0
- joint RL_calf_joint: origin xyz=0 0 -0.2115 rpy=0 0 0 -> xyz=0 0.07125 -0.21183 rpy=0 -0.98 0
- joint RL_foot_fixed: origin xyz=0 0 -0.23039 rpy=0 0 0 -> xyz=0 0 -0.240 rpy=0 0 0
- joint RL_hip_joint: origin xyz=-0.1305 0.05 0 rpy=0 0 0 -> xyz=-0.130 0.05 0 rpy=0 0 0
- joint RL_thigh_joint: origin xyz=0 0.077476 0 rpy=0 0 0 -> xyz=-0.06 0.015 0 rpy=0 0 0
- joint RR_calf_joint: origin xyz=0 0 -0.2115 rpy=0 0 0 -> xyz=0 -0.07125 -0.21183 rpy=0 -0.98 0
- joint RR_foot_fixed: origin xyz=0 0 -0.23039 rpy=0 0 0 -> xyz=0 0 -0.240 rpy=0 0 0
- joint RR_thigh_joint: origin xyz=0 -0.077476 0 rpy=0 0 0 -> xyz=-0.06 -0.015 0 rpy=0 0 0
